Commit message: Remove external dependency on kobuki_description Fix left wheel radius. Fix ros_diff_drive plugin warnings

File: urdf/turtlebot2.urdf (robot description, URDF)
Before this commit: robot turtlebot, 36 links, 35 joints
Links:
- link base_link: geometry collision cylinder length=0.10938 radius=0.178; visual mesh filename=package://ekf_ukf/urdf/meshes/main_body.dae
- link camera_link: geometry collision box size=0.0730 0.2760 0.0720; visual mesh filename=package://ekf_ukf/urdf/meshes/stacks/hexagons/xtion_pro_cam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
- link mount_asus_xtion_pro_link: geometry collision box size=0.0330 0.2760 0.0120; visual mesh filename=package://ekf_ukf/urdf/meshes/stacks/hexagons/xtion_pro_sta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
- link plate_bottom_link: geometry collision cylinder length=0.006 radius=0.170; visual mesh filename=package://ekf_ukf/urdf/meshes/stacks/hexagons/plate_bottom.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
- link plate_middle_link: geometry collision cylinder length=0.006 radius=0.170; visual mesh filename=package://ekf_ukf/urdf/meshes/stacks/hexagons/plate_middle.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
- link plate_top_link: geometry collision cylinder length=0.006 radius=0.170; visual mesh filename=package://ekf_ukf/urdf/meshes/stacks/hexagons/plate_top.dae
- link pole_bottom_0_link: geometry collision cylinder length=0.0492 radius=0.006; visual mesh filename=package://ekf_ukf/urdf/meshes/stacks/hexagons/pole_bottom.d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
- link pole_bottom_1_link: geometry collision cylinder length=0.0492 radius=0.006; visual mesh filename=package://ekf_ukf/urdf/meshes/stacks/hexagons/pole_bottom.d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
- link pole_bottom_2_link: geometry collision cylinder length=0.0492 radius=0.006; visual mesh filename=package://ekf_ukf/urdf/meshes/stacks/hexagons/pole_bottom.d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
- link pole_bottom_3_link: geometry collision cylinder length=0.0492 radius=0.006; visual mesh filename=package://ekf_ukf/urdf/meshes/stacks/hexagons/pole_bottom.d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
- link pole_bottom_4_link: geometry collision cylinder length=0.0492 radius=0.006; visual mesh filename=package://ekf_ukf/urdf/meshes/stacks/hexagons/pole_bottom.d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
- link pole_bottom_5_link: geometry collision cylinder length=0.0492 radius=0.006; visual mesh filename=package://ekf_ukf/urdf/meshes/stacks/hexagons/pole_bottom.d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
- link pole_kinect_0_link: geometry collision cylinder length=0.0936 radius=0.006; visual mesh filename=package://ekf_ukf/urdf/meshes/stacks/hexagons/sensor_pole.d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
- link pole_kinect_1_link: geometry collision cylinder length=0.0936 radius=0.006; visual mesh filename=package://ekf_ukf/urdf/meshes/stacks/hexagons/sensor_pole.d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
- link pole_middle_0_link: geometry collision cylinder length=0.0608 radius=0.006; visual mesh filename=package://ekf_ukf/urdf/meshes/stacks/hexagons/pole_middle.d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
- link pole_middle_1_link: geometry collision cylinder length=0.0608 radius=0.006; visual mesh filename=package://ekf_ukf/urdf/meshes/stacks/hexagons/pole_middle.d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
- link pole_middle_2_link: geometry collision cylinder length=0.0608 radius=0.006; visual mesh filename=package://ekf_ukf/urdf/meshes/stacks/hexagons/pole_middle.d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
- link pole_middle_3_link: geometry collision cylinder length=0.0608 radius=0.006; visual mesh filename=package://ekf_ukf/urdf/meshes/stacks/hexagons/pole_middle.d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
- link pole_top_0_link: geometry collision cylinder length=0.2032 radius=0.006; visual mesh filename=package://ekf_ukf/urdf/meshes/stacks/hexagons/pole_top.dae
- link pole_top_1_link: geometry collision cylinder length=0.2032 radius=0.006; visual mesh filename=package://ekf_ukf/urdf/meshes/stacks/hexagons/pole_top.dae
- link pole_top_2_link: geometry collision cylinder length=0.2032 radius=0.006; visual mesh filename=package://ekf_ukf/urdf/meshes/stacks/hexagons/pole_top.dae
- link pole_top_3_link: geometry collision cylinder length=0.2032 radius=0.006; visual mesh filename=package://ekf_ukf/urdf/meshes/stacks/hexagons/pole_top.dae
- link wheel_left_link: geometry collision cylinder length=0.0206 radius=0.0350; visual mesh filename=package://ekf_ukf/urdf/meshes/wheel.dae
- link wheel_right_link: geometry collision cylinder length=0.0206 radius=0.0350; visual mesh filename=package://ekf_ukf/urdf/meshes/wheel.dae

Commit message: Fix issue transparent robot model in 'Ros Development Studio' Revert 'Remove external dependency on kobuki_description' Fix ressource not found on kobuki_description pkg (move meshes to urdf/sensors/)

File: urdf/turtlebot2.urdf (robot description, URDF)
Before this commit: robot turtlebot, 36 links, 35 joints
Links:
- link base_link: geometry collision cylinder length=0.10938 radius=0.178; visual mesh filename=package://kobuki_description/meshes/main_body.dae
- link camera_link: geometry collision box size=0.0730 0.2760 0.0720; visual mesh filename=package://kobuki_description/meshes/sensors/xtion_pro_camer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
- link laser_sensor_link: geometry collision box size=0.1 0.1 0.1; visual mesh filename=package://particle_filter/models/hokuyo/meshes/hokuyo.dae
- link mount_asus_xtion_pro_link: geometry collision box size=0.0330 0.2760 0.0120; visual mesh filename=package://kobuki_description/meshes/sensors/xtion_pro_stack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
- link plate_bottom_link: geometry collision cylinder length=0.006 radius=0.170; visual mesh filename=package://kobuki_description/meshes/stacks/hexagons/plate_b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
- link plate_middle_link: geometry collision cylinder length=0.006 radius=0.170; visual mesh filename=package://kobuki_description/meshes/stacks/hexagons/plate_m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
- link plate_top_link: geometry collision cylinder length=0.006 radius=0.170; visual mesh filename=package://kobuki_description/meshes/stacks/hexagons/plate_t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
- link pole_bottom_0_link: geometry collision cylinder length=0.0492 radius=0.006; visual mesh filename=package://kobuki_description/meshes/stacks/hexagons/pole_bo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
- link pole_bottom_1_link: geometry collision cylinder length=0.0492 radius=0.006; visual mesh filename=package://kobuki_description/meshes/stacks/hexagons/pole_bo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
- link pole_bottom_2_link: geometry collision cylinder length=0.0492 radius=0.006; visual mesh filename=package://kobuki_description/meshes/stacks/hexagons/pole_bo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
- link pole_bottom_3_link: geometry collision cylinder length=0.0492 radius=0.006; visual mesh filename=package://kobuki_description/meshes/stacks/hexagons/pole_bo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
- link pole_bottom_4_link: geometry collision cylinder length=0.0492 radius=0.006; visual mesh filename=package://kobuki_description/meshes/stacks/hexagons/pole_bo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
- link pole_bottom_5_link: geometry collision cylinder length=0.0492 radius=0.006; visual mesh filename=package://kobuki_description/meshes/stacks/hexagons/pole_bo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
- link pole_kinect_0_link: geometry collision cylinder length=0.0936 radius=0.006; visual mesh filename=package://kobuki_description/meshes/sensors/sensor_pole.dae
- link pole_kinect_1_link: geometry collision cylinder length=0.0936 radius=0.006; visual mesh filename=package://kobuki_description/meshes/sensors/sensor_pole.dae
- link pole_middle_0_link: geometry collision cylinder length=0.0608 radius=0.006; visual mesh filename=package://kobuki_description/meshes/stacks/hexagons/pole_mi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
- link pole_middle_1_link: geometry collision cylinder length=0.0608 radius=0.006; visual mesh filename=package://kobuki_description/meshes/stacks/hexagons/pole_mi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
- link pole_middle_2_link: geometry collision cylinder length=0.0608 radius=0.006; visual mesh filename=package://kobuki_description/meshes/stacks/hexagons/pole_mi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
- link pole_middle_3_link: geometry collision cylinder length=0.0608 radius=0.006; visual mesh filename=package://kobuki_description/meshes/stacks/hexagons/pole_mi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
- link pole_top_0_link: geometry collision cylinder length=0.2032 radius=0.006; visual mesh filename=package://kobuki_description/meshes/stacks/hexagons/pole_to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
- link pole_top_1_link: geometry collision cylinder length=0.2032 radius=0.006; visual mesh filename=package://kobuki_description/meshes/stacks/hexagons/pole_to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
- link pole_top_2_link: geometry collision cylinder length=0.2032 radius=0.006; visual mesh filename=package://kobuki_description/meshes/stacks/hexagons/pole_to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
- link pole_top_3_link: geometry collision cylinder length=0.2032 radius=0.006; visual mesh filename=package://kobuki_description/meshes/stacks/hexagons/pole_to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
- link wheel_left_link: geometry collision cylinder length=0.0206 radius=0.0350; visual mesh filename=package://kobuki_description/meshes/wheel.dae
- link wheel_right_link: geometry collision cylinder length=0.0206 radius=0.0350; visual mesh filename=package://kobuki_description/meshes/wheel.dae
